File: MotorMonster/Drivers.kicad_sch (KiCad schematic)
At the start: 39 parts

Commit message: basic layout and some routing done
Parts:
- added NT1, NT2: NetTie_2, NetTie:NetTie-2_SMD_Pad0.5mm, symbol Device:NetTie_2
Connections:
- net GND: now also NT1.2, NT2.2; no longer R_S107.2, R_S113.2
- net S1B_Ret: now reaches Q_S103.1 (D), Q_S103.2 (G), Q_S103.3 (S), Q_S104.1 (D), Q_S104.2 (G), Q_S104.3 (S), R_S106.2, R_S1B1.1, R_S1B2.1
- net S1A_Ret: now reaches Q_S107.1 (D), Q_S107.2 (G), Q_S107.3 (S), Q_S108.1 (D), Q_S108.2 (G), Q_S108.3 (S), R_S112.2, R_S1A1.1, R_S1A2.1
- new net: NT2.1, R_S113.2
- new net: NT1.1, R_S107.2
Changed lines of the file:
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@@
 	(wire
 		(pts
-			(xy 160.02 97.79) (xy 170.18 97.79)
-		)
-		(stroke
-			(width 0)
-			(type default)
-		)
-	)
-	(wire
-		(pts
 			(xy 167.64 62.23) (xy 167.64 66.04)
 		)
@@
 	(wire
 		(pts
-			(xy 170.18 163.83) (xy 180.34 163.83)
+			(xy 171.45 163.83) (xy 180.34 163.83)
 		)
 		(stroke
@@
 	(wire
 		(pts
-			(xy 170.18 92.71) (xy 180.34 92.71)
+			(xy 171.45 92.71) (xy 180.34 92.71)
 		)
 		(stroke
@@
 	(wire
 		(pts
+			(xy 168.91 97.79) (xy 171.45 97.79)
+		)
+		(stroke
+			(width 0)
+			(type default)
+		)
+	)
+	(wire
+		(pts
 			(xy 86.36 36.83) (xy 86.36 38.1)
 		)
@@
 	(wire
 		(pts
-			(xy 170.18 168.91) (xy 170.18 163.83)
+			(xy 171.45 168.91) (xy 171.45 163.83)
 		)
 		(stroke
@@
 	(wire
 		(pts
-			(xy 160.02 168.91) (xy 170.18 168.91)
+			(xy 168.91 168.91) (xy 171.45 168.91)
 		)
 		(stroke
@@
 	(wire
 		(pts
+			(xy 160.02 168.91) (xy 163.83 168.91)
+		)
+		(stroke
+			(width 0)
+			(type default)
+		)
+	)
+	(wire
+		(pts
 			(xy 185.42 156.21) (xy 198.12 156.21)
 		)
@@
 	(wire
 		(pts
-			(xy 170.18 97.79) (xy 170.18 92.71)
+			(xy 171.45 97.79) (xy 171.45 92.71)
 		)
 		(stroke
@@
 	(wire
 		(pts
+			(xy 160.02 97.79) (xy 163.83 97.79)
+		)
+		(stroke
+			(width 0)
+			(type default)
+		)
+	)
+	(wire
+		(pts
 			(xy 167.64 133.35) (xy 167.64 137.16)
 		)
@@
 		)
 	)
+	(global_label "S1B_Ret"
+		(shape input)
+		(at 200.66 85.09 0)
+		(fields_autoplaced yes)
+		(effects
+			(font
+				(size 1.27 1.27)
+			)
+			(justify left)
+		)
+		(property "Intersheetrefs" "${INTERSHEET_REFS}"
+			(at 211.3861 85.09 0)
+			(effects
+				(font
+					(size 1.27 1.27)
+				)
+				(justify left)
+				(hide yes)
+			)
+		)
+	)
 	(global_label "1B+"
 		(shape input)
@@
 		)
 	)
+	(global_label "S1A_Ret"
+		(shape input)
+		(at 200.66 156.21 0)
+		(fields_autoplaced yes)
+		(effects
+			(font
+				(size 1.27 1.27)
+			)
+			(justify left)
+		)
+		(property "Intersheetrefs" "${INTERSHEET_REFS}"
+			(at 211.2047 156.21 0)
+			(effects
+				(font
+					(size 1.27 1.27)
+				)
+				(justify left)
+				(hide yes)
+			)
+		)
+	)
 	(global_label "1A-"
 		(shape input)
@@
 	)
 	(symbol
+		(lib_id "Device:NetTie_2")
+		(at 166.37 168.91 0)
+		(unit 1)
+		(exclude_from_sim no)
+		(in_bom no)
+		(on_board yes)
+		(dnp no)
+		(fields_autoplaced yes)
+		(property "Reference" "NT2"
+			(at 166.37 163.83 0)
+			(effects
+				(font
+					(size 1.27 1.27)
+				)
+			)
+		)
+		(property "Value" "NetTie_2"
+			(at 166.37 166.37 0)
+			(effects
+				(font
+					(size 1.27 1.27)
+				)
+			)
+		)
+		(property "Footprint" "NetTie:NetTie-2_SMD_Pad0.5mm"
+			(at 166.37 168.91 0)
+			(effects
+				(font
+					(size 1.27 1.27)
+				)
+				(hide yes)
+			)
+		)
+		(property "Datasheet" "~"
+			(at 166.37 168.91 0)
+			(effects
+				(font
+					(size 1.27 1.27)
+				)
+				(hide yes)
+			)
+		)
+		(property "Description" "Net tie, 2 pins"
+			(at 166.37 168.91 0)
+			(effects
+				(font
+					(size 1.27 1.27)
+				)
+				(hide yes)
+			)
+		)
+		(pin "1"
+		)
+		(pin "2"
+		)
+		(instances
+			(project ""
+				(path "/798975c2-d104-4b51-bc9d-eb81d8f1bd39/41de1745-7488-4e44-91c5-64997c6fd692"
+					(reference "NT2")
+					(unit 1)
+				)
+			)
+		)
+	)
+	(symbol
 		(lib_id "power:+3V3")
 		(at 57.15 66.04 0)
@@
 					(unit 1)
 				)
+			)
+		)
+	)
+	(symbol
+		(lib_id "Device:NetTie_2")
+		(at 166.37 97.79 0)
+		(unit 1)
+		(exclude_from_sim no)
+		(in_bom no)
+		(on_board yes)
+		(dnp no)
+		(fields_autoplaced yes)
+		(property "Reference" "NT1"
+			(at 166.37 92.71 0)
+			(effects
+				(font
+					(size 1.27 1.27)
+				)
+			)
+		)
+		(property "Value" "NetTie_2"
+			(at 166.37 95.25 0)
+			(effects
+				(font
+					(size 1.27 1.27)
+				)
+			)
+		)
+		(property "Footprint" "NetTie:NetTie-2_SMD_Pad0.5mm"
+			(at 166.37 97.79 0)
+			(effects
+				(font
+					(size 1.27 1.27)
+				)
+				(hide yes)
+			)
+		)
+		(property "Datasheet" "~"
+			(at 166.37 97.79 0)
+			(effects
+				(font
+					(size 1.27 1.27)
+				)
+				(hide yes)
+			)
+		)
+		(property "Description" "Net tie, 2 pins"
+			(at 166.37 97.79 0)
+			(effects
+				(font
+					(size 1.27 1.27)
+				)
+				(hide yes)
+			)
+		)
+		(pin "1"
+		)
+		(pin "2"
+		)
+		(instances
+			(project ""
+				(path "/798975c2-d104-4b51-bc9d-eb81d8f1bd39/41de1745-7488-4e44-91c5-64997c6fd692"
+					(reference "NT1")
+					(unit 1)
+				)

Commit message: fully laid out
Parts:
- removed R_S1A2, R_S1B2: R, Resistor_SMD:R_2512_6332Metric_Pad1.40x3.35mm_HandSolder, symbol Device:R_Small
- added J4: Conn_01x04, Connector_JST:JST_XH_B4B-XH-A_1x04_P2.50mm_Vertical, symbol Connector_Generic:Conn_01x04
Connections:
- net 1A+: now also J4.1 (Pin_1)
- net 1A-: now also J4.2 (Pin_2)
- net 1B+: now also J4.4 (Pin_4)
- net 1B-: now also J4.3 (Pin_3)
Other:
- moved on the sheet: R_S1A1, R_S1B1
