File: MotorMonster/MotorMonster.kicad_sch (KiCad schematic)
At the start: 45 parts, among them J1 USB C Connector, J2 JTAG_TC2030, J3 HV In, SW1 Boot, U1 XC6206, U2 USBLC6-2SC6, U3 RP2040, U4 W25Q128JVS, U5 LM5164DDA, Y1 12MHz

Commit message: basic layout and some routing done
Parts:
- removed D1: Schottky Diode, Diode_SMD:D_SOD-123, symbol Device:D_Small
Connections:
- net +3V3: now also U1.2 (VO)
- net GND: now also J3.1 (Pin_1); no longer J3.2 (Pin_2)
- net Vh: now reaches F2.1
- net Vh: now also J3.2 (Pin_2); no longer J3.1 (Pin_1)
Other:
- moved on the sheet: F2, J3
Changed lines of the file:
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@@
 	)
 	(junction
+		(at 219.71 83.82)
+		(diameter 0)
+		(color 0 0 0 0)
+	)
+	(junction
 		(at 250.19 148.59)
 		(diameter 0)
@@
 	)
 	(junction
-		(at 173.99 87.63)
+		(at 74.93 171.704)
 		(diameter 0)
 		(color 0 0 0 0)
 	)
 	(junction
-		(at 74.93 171.704)
+		(at 173.99 87.63)
 		(diameter 0)
 		(color 0 0 0 0)
@@
 	(wire
 		(pts
-			(xy 227.33 83.82) (xy 236.22 83.82)
+			(xy 229.87 83.82) (xy 236.22 83.82)
 		)
 		(stroke
@@
 	(wire
 		(pts
+			(xy 219.71 83.82) (xy 224.79 83.82)
+		)
+		(stroke
+			(width 0)
+			(type default)
+		)
+	)
+	(wire
+		(pts
 			(xy 151.765 125.73) (xy 156.845 125.73)
 		)
@@
 	(wire
 		(pts
+			(xy 219.71 86.36) (xy 222.25 86.36)
+		)
+		(stroke
+			(width 0)
+			(type default)
+		)
+	)
+	(wire
+		(pts
 			(xy 48.26 187.96) (xy 48.26 186.69)
 		)
@@
 		)
 	)
+	(wire
+		(pts
+			(xy 168.91 87.63) (xy 173.99 87.63)
+		)
+		(stroke
+			(width 0)
+			(type default)
+		)
+	)
 	(bus
 		(pts
@@
 	(wire
 		(pts
-			(xy 219.71 83.82) (xy 222.25 83.82)
-		)
-		(stroke
-			(width 0)
-			(type default)
-		)
-	)
-	(wire
-		(pts
 			(xy 122.555 184.15) (xy 113.665 184.15)
 		)
@@
 	(wire
 		(pts
+			(xy 219.71 78.74) (xy 219.71 83.82)
+		)
+		(stroke
+			(width 0)
+			(type default)
+		)
+	)
+	(wire
+		(pts
 			(xy 195.58 142.24) (xy 204.47 142.24)
 		)
@@
 		)
 	)
+	(global_label "Vh"
+		(shape input)
+		(at 219.71 78.74 180)
+		(fields_autoplaced yes)
+		(effects
+			(font
+				(size 1.27 1.27)
+			)
+			(justify right)
+		)
+		(property "Intersheetrefs" "${INTERSHEET_REFS}"
+			(at 214.4872 78.74 0)
+			(effects
+				(font
+					(size 1.27 1.27)
+				)
+				(justify right)
+				(hide yes)
+			)
+		)
+	)
 	(global_label "XTAL_IN"
 		(shape input)
@@
 		(lib_name "GND_3")
 		(lib_id "power:GND")
-		(at 219.71 86.36 0)
+		(at 222.25 86.36 0)
 		(unit 1)
 		(exclude_from_sim no)
@@
 		(fields_autoplaced yes)
 		(property "Reference" "#PWR052"
-			(at 219.71 92.71 0)
+			(at 222.25 92.71 0)
 			(effects
 				(font
@@
 		)
 		(property "Value" "GND"
-			(at 219.71 91.44 0)
+			(at 222.25 91.44 0)
 			(effects
 				(font
@@
 		)
 		(property "Footprint" ""
-			(at 219.71 86.36 0)
+			(at 222.25 86.36 0)
 			(effects
 				(font
@@
 		)
 		(property "Datasheet" ""
-			(at 219.71 86.36 0)
+			(at 222.25 86.36 0)
 			(effects
 				(font
@@
 		)
 		(property "Description" "Power symbol creates a global label with name \"GND\" , ground"
-			(at 219.71 86.36 0)
+			(at 222.25 86.36 0)
 			(effects
 				(font
@@
 	)
 	(symbol
-		(lib_id "Device:D_Small")
-		(at 171.45 87.63 180)
-		(unit 1)
-		(exclude_from_sim no)
-		(in_bom yes)
-		(on_board yes)
-		(dnp no)
-		(property "Reference" "D1"
-			(at 174.8028 79.883 0)
-			(effects
-				(font
-					(size 1.27 1.27)
-				)
-			)
-		)
-		(property "Value" "Schottky Diode"
-			(at 174.8028 82.423 0)
-			(effects
-				(font
-					(size 1.27 1.27)
-				)
-			)
-		)
-		(property "Footprint" "Diode_SMD:D_SOD-123"
-			(at 171.45 87.63 90)
-			(effects
-				(font
-					(size 1.27 1.27)
-				)
-				(hide yes)
-			)
-		)
-		(property "Datasheet" "~"
-			(at 171.45 87.63 90)
-			(effects
-				(font
-					(size 1.27 1.27)
-				)
-				(hide yes)
-			)
-		)
-		(property "Description" ""
-			(at 171.45 87.63 0)
-			(effects
-				(font
-					(size 1.27 1.27)
-				)
-				(hide yes)
-			)
-		)
-		(property "LCSC" "C8598"
-			(at 171.45 87.63 0)
-			(effects
-				(font
-					(size 1.27 1.27)
-				)
-				(hide yes)
-			)
-		)
-		(pin "1"
-		)
-		(pin "2"
-		)
-		(instances
-			(project "OpenRectangle"
-				(path "/0ee7bd02-e26d-4978-ae8c-675a718c78c0"
-					(reference "D1")
-					(unit 1)
-				)
-			)
-			(project "OpenRectangleTemplate"
-				(path "/798975c2-d104-4b51-bc9d-eb81d8f1bd39"
-					(reference "D1")
-					(unit 1)
-				)
-			)
-		)
-	)
-	(symbol
 		(lib_id "Device:C_Small")
 		(at 57.15 184.15 0)
@@
 	(symbol
 		(lib_id "Connector:Screw_Terminal_01x02")
-		(at 214.63 83.82 0)
-		(mirror y)
+		(at 214.63 86.36 180)
 		(unit 1)
 		(exclude_from_sim no)
@@
 		(dnp no)
 		(property "Reference" "J3"
-			(at 212.09 83.8199 0)
+			(at 212.09 86.3601 0)
 			(effects
 				(font
@@
 		)
 		(property "Value" "HV In"
-			(at 212.09 86.3599 0)
+			(at 212.09 83.8201 0)
 			(effects
 				(font
@@
 		)
 		(property "Footprint" "TerminalBlock:TerminalBlock_Altech_AK300-2_P5.00mm"
-			(at 214.63 83.82 0)
+			(at 214.63 86.36 0)
 			(effects
 				(font
@@
 		)
 		(property "Datasheet" "~"
-			(at 214.63 83.82 0)
+			(at 214.63 86.36 0)
 			(effects
 				(font
@@
 		)
 		(property "Description" "CUI Devices TB010-508-02BE"
-			(at 214.63 83.82 0)
+			(at 214.63 86.36 0)
 			(effects
 				(font
@@
 		(lib_name "Fuse_Small_1")
 		(lib_id "Device:Fuse_Small")
-		(at 224.79 83.82 0)
+		(at 227.33 83.82 0)
 		(unit 1)
 		(exclude_from_sim no)
@@
 		(fields_autoplaced yes)
 		(property "Reference" "F2"
-			(at 224.79 78.74 0)
+			(at 227.33 78.74 0)
 			(effects
 				(font
@@
 		)
 		(property "Value" "Fuse_Small"
-			(at 224.79 81.28 0)
+			(at 227.33 81.28 0)
 			(effects
 				(font
@@
 		)
 		(property "Footprint" "Fuse:Fuseholder_Clip-6.3x32mm_Littelfuse_122_Inline_P34.21x7.62mm_D2.54mm_Horizontal"
-			(at 224.79 83.82 0)
+			(at 227.33 83.82 0)
 			(effects
 				(font
@@
 		)
 		(property "Datasheet" "~"
-			(at 224.79 83.82 0)
+			(at 227.33 83.82 0)
 			(effects
 				(font
@@
 		)
 		(property "Description" "Littelfuse 01220083"
-			(at 224.79 83.82 0)
+			(at 227.33 83.82 0)
 			(effects
 				(font

Commit message: fully laid out
Parts:
- removed J1: USB C Connector, footprints:TYPE-C_24P_QCHT, symbol Connector:USB_C_Receptacle
- added P1: USB_C_Plug_USB2.0, Connector_USB:USB_C_Receptacle_G-Switch_GT-USB-7010ASV, symbol Connector:USB_C_Receptacle_USB2.0_16P
Connections:
- net DBUS+: now also P1.A6 (D+), P1.B6 (D+)
- net DBUS-: now also P1.A7 (D-), P1.B7 (D-)
- net GND: now also P1.A1 (GND), P1.A12 (GND), P1.B1 (GND), P1.B12 (GND)
- net S1CS: now also U3.8 (GPIO6); no longer U3.7 (GPIO5)
- net Vbus: now also P1.A4 (VBUS), P1.A9 (VBUS), P1.B4 (VBUS), P1.B9 (VBUS)
- net S1En: now reaches U3.2 (GPIO0)
- net S1Dir: now reaches U3.3 (GPIO1)
- net at R2.2: now also P1.B5 (CC2)
- net at R3.1: now also P1.A5 (CC1)
- net at R1.2: now also P1.S1 (SHIELD)
- new net S1Step: U3.7 (GPIO5)
- no-connect marks 10 -> 2
Other:
- moved on the sheet: F1, R1, R2, R3
